File: Klask_PCB.kicad_pcb (KiCad board)
At the start: 2 copper layers, 69.1 x 53.8 mm, 10 parts, among them SW1 SW_Push_SPDT

Commit message: update
Parts:
- added J1: Conn_01x02_Socket, TerminalBlock:TerminalBlock_Xinya_XY308-2.54-2P_1x02_P2.54mm_Horizontal, F.Cu at (91.4, 80.0)
- added J2: Conn_01x02_Socket, TerminalBlock:TerminalBlock_Xinya_XY308-2.54-2P_1x02_P2.54mm_Horizontal, F.Cu at (99.1, 80.0)
- added J3: Conn_01x02_Socket, TerminalBlock:TerminalBlock_Xinya_XY308-2.54-2P_1x02_P2.54mm_Horizontal, F.Cu at (141.0, 50.8)
- added J4: Conn_01x02_Socket, TerminalBlock:TerminalBlock_Xinya_XY308-2.54-2P_1x02_P2.54mm_Horizontal, F.Cu at (141.0, 58.4)
- added R3: 1k, Resistor_THT:R_Box_L8.4mm_W2.5mm_P5.08mm, F.Cu at (87.6, 58.4)
- added R4: 1k, Resistor_THT:R_Box_L8.4mm_W2.5mm_P5.08mm, F.Cu at (87.6, 48.3)
- added SW2: SW_Push_SPDT, TerminalBlock:TerminalBlock_Xinya_XY308-2.54-2P_1x02_P2.54mm_Horizontal, F.Cu at (82.5, 52.1)
- added SW3: SW_Push_SPDT, TerminalBlock:TerminalBlock_Xinya_XY308-2.54-2P_1x02_P2.54mm_Horizontal, F.Cu at (82.5, 41.9)
- moved D1 26.5 mm to (81.3, 68.6)
- moved R1 20.6 mm to (90.2, 71.1), turned to 180 degrees
- moved R2 19.6 mm to (87.6, 67.3), turned to 0 degrees
- moved C1 15.3 mm to (87.6, 63.5), turned to 0 degrees
- moved SW1 14.0 mm to (83.8, 80.0), turned to 0 degrees
- moved C4 11.5 mm to (132.1, 61.0), turned to 180 degrees
- moved C3 8.21 mm to (110.5, 61.0), turned to 180 degrees
- moved A2 4.26 mm to (114.3, 55.9)
- moved A1 1.80 mm to (92.7, 55.9)
Connections:
- A3 pad 26: unconnected-(A3-D11-Pad26) -> /SW_X
- A3 pad 27: unconnected-(A3-D12-Pad27) -> /SW_Y
- A3 pad 4: unconnected-(A3-3V3-Pad4) -> /3V3
Routing:
- net /nEN: track 61.4 -> 0.00 mm
- net /A0: track 45.4 -> 0.00 mm
- net /M2: track 42.7 -> 0.00 mm
- net /M1: track 42.7 -> 0.00 mm
- net /M0: track 42.5 -> 0.00 mm
- net /MX_A1: track 0.00 -> 34.4 mm
- net /MX_STEP: track 31.4 -> 0.00 mm
- net /MX_DIR: track 30.1 -> 0.00 mm
- net /MY_B1: track 0.00 -> 29.1 mm
- net /MY_A2: track 0.00 -> 26.2 mm
- net /MX_B2: track 0.00 -> 25.7 mm
- net /MX_B1: track 0.00 -> 25.7 mm
- net /MX_A2: track 0.00 -> 25.7 mm
- net /MY_A1: track 0.00 -> 23.7 mm
- net /MY_STEP: track 18.1 -> 0.00 mm
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
Commit message: update
Parts:
- removed R3, R4: 1k, Resistor_THT:R_Box_L8.4mm_W2.5mm_P5.08mm
- removed SW1: SW_Push_SPDT, TerminalBlock:TerminalBlock_Xinya_XY308-2.54-2P_1x02_P2.54mm_Horizontal
- added SW4: SW_Push, TerminalBlock:TerminalBlock_Xinya_XY308-2.54-2P_1x02_P2.54mm_Horizontal, F.Cu at (83.6, 37.1)
- added SW5: SW_Push, TerminalBlock:TerminalBlock_Xinya_XY308-2.54-2P_1x02_P2.54mm_Horizontal, F.Cu at (90.7, 37.1)
- added SW6: SW_Push, TerminalBlock:TerminalBlock_Xinya_XY308-2.54-2P_1x02_P2.54mm_Horizontal, F.Cu at (84.3, 80.0)
- D1: footprint LED_THT:LED_D2.0mm_W4.8mm_H2.5mm_FlatTop -> LED_THT:LED_D3.0mm
- R1: value 3.3K -> 510
- R2: value 1K -> 180
- SW2, SW3: value SW_Push_SPDT -> SW_Push
- moved SW3 7.87 mm to (82.8, 49.8)
- moved SW2 4.58 mm to (82.8, 56.6)
- moved C1 0.57 mm to (87.9, 64.0)
- moved R2 0.36 mm to (87.9, 67.6)
- moved R1 0.26 mm to (90.4, 71.1)
- moved A1 0.25 mm to (93.0, 55.9)
- moved C3 0.25 mm to (110.7, 61.0)
Connections:
- A3 pad 18: /MY_STEP -> /nEN
- A3 pad 19: /MY_DIR -> /MY_STEP
- A3 pad 20: unconnected-(A3-D5-Pad20) -> /MY_DIR
- A3 pad 22: /nEN -> unconnected-(A3-D7-Pad22)
- A3 pad 26: /SW_X -> unconnected-(A3-D11-Pad26)
- A3 pad 27: /SW_Y -> /SW_A
- A3 pad 28: unconnected-(A3-D13-Pad28) -> /SW_B
- A3 pad 31: unconnected-(A3-SDA/A4-Pad31) -> /SW_X
- A3 pad 32: unconnected-(A3-SCL/A5-Pad32) -> /SW_Y
- J1 pad 1: /MX_A1 -> /MX_A2
- J1 pad 2: /MX_A2 -> /MX_A1
- J4 pad 1: /MY_B1 -> /MY_B2
- J4 pad 2: /MY_B2 -> /MY_B1
- SW2 pad 1: unconnected-(SW2-A-Pad1) -> /SW_A
- SW2 pad 2: Net-(SW2-B) -> GND
- SW3 pad 1: unconnected-(SW3-A-Pad1) -> /SW_B
- SW3 pad 2: Net-(SW3-B) -> GND
Routing:
- net /A0: track 0.00 -> 60.2 mm
- net /nEN: track 0.00 -> 43.9 mm
- net /M2: track 0.00 -> 41.5 mm
- net /M1: track 0.00 -> 41.2 mm
- net /SW_A: track 0.00 -> 40.9 mm
- net /M0: track 0.00 -> 39.8 mm
- net /SW_B: track 0.00 -> 30.8 mm
- net /MX_STEP: track 0.00 -> 28.3 mm
- net /MX_DIR: track 0.00 -> 28.3 mm
- net /MY_STEP: track 0.00 -> 18.4 mm
- net /MY_DIR: track 0.00 -> 18.4 mm
- net /SW_X: track 0.00 -> 18.2 mm
- net /MY_B1: track 29.1 -> 20.9 mm
- net /MX_A1: track 34.4 -> 26.9 mm
- net /SW_Y: track 0.00 -> 7.49 mm
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
Commit message: update
Parts:
- moved D1 0.25 mm to (81.0, 68.6)
Changed lines of the file:
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@@
 	(footprint "LED_THT:LED_D3.0mm"
 		(layer "F.Cu")
-		(at 81.28 68.58 -90)
+		(at 81.026 68.58 -90)
 		(descr "LED, diameter 3.0mm, 2 pins, generated by kicad-footprint-generator")
 		(tags "LED")
 		(property "Reference" "D1"
-			(at 1.27 -2.96 270)
+			(at -2.032 0 270)
 			(layer "F.SilkS")
 			(effects
@@
 	)
 	(segment
-		(start 86.868 68.58)
-		(end 87.884 67.564)
+		(start 111.764 39.116)
+		(end 115.32 35.56)
 		(width 0.2)
 		(layer "F.Cu")
@@
 	)
 	(segment
-		(start 111.764 39.116)
-		(end 115.32 35.56)
+		(start 87.884 64.008)
+		(end 88.87 63.022)
 		(width 0.2)
 		(layer "F.Cu")
@@
 	)
 	(segment
-		(start 87.884 64.008)
-		(end 88.87 63.022)
+		(start 86.868 68.58)
+		(end 87.884 67.564)
 		(width 0.2)
 		(layer "F.Cu")
@@
 	)
 	(segment
-		(start 81.28 68.58)
-		(end 86.868 68.58)
+		(start 88.87 45.242)
+		(end 94.996 39.116)
 		(width 0.2)
 		(layer "F.Cu")
@@
 	)
 	(segment
-		(start 88.87 45.242)
-		(end 94.996 39.116)
+		(start 81.026 68.58)
+		(end 86.868 68.58)
 		(width 0.2)
 		(layer "F.Cu")
@@
 	(segment
 		(start 85.085 71.12)
-		(end 81.28 71.12)
+		(end 81.026 71.12)
 		(width 0.2)
 		(layer "F.Cu")

Commit message: update
Parts:
- removed SW6: SW_Push, TerminalBlock:TerminalBlock_Xinya_XY308-2.54-2P_1x02_P2.54mm_Horizontal
- added J5: Conn_01x02_Socket, TerminalBlock:TerminalBlock_Xinya_XY308-2.54-2P_1x02_P2.54mm_Horizontal, F.Cu at (84.3, 80.0)
- moved SW5 7.01 mm to (85.9, 42.2), turned to -90 degrees
- moved SW3 3.11 mm to (85.9, 49.0)
- moved SW2 3.11 mm to (85.9, 55.9)
- moved SW4 2.75 mm to (85.9, 35.6), turned to -90 degrees
Connections:
- A1 pad 8: /v_motor -> +12V
- A2 pad 8: /v_motor -> +12V
- A3 pad 31: /SW_X -> /SW_Y
- A3 pad 32: /SW_Y -> /SW_X
- C3 pad 1: /v_motor -> +12V
- C4 pad 1: /v_motor -> +12V
- R1 pad 1: /v_motor -> +12V
Routing:
- net /v_motor: track 94.3 -> 0.00 mm
- net +12V: track 0.00 -> 94.3 mm
- net /SW_Y: track 7.49 -> 17.0 mm
- net /SW_X: track 18.2 -> 11.7 mm
- net /SW_A: track 40.9 -> 37.6 mm
- net /SW_B: track 30.8 -> 28.5 mm
- net GND: vias 0 -> 26
Other:
- outline, holes or cut-outs redrawn
- board text added: "CoreXY 3.3V v0.1.0 by motty"
- board text added: "MX_A"
- board text added: "MX_B"
- board text added: "MY_A"
- board text added: "MY_B"
- board text added: "SW_X"
- board text added: "SW_Y"
- board text added: "v12"
