File: Klask_PCB.kicad_pcb (KiCad board)
At the start: 2 copper layers, 69.1 x 53.8 mm, 18 parts, among them J1 Conn_01x02_Socket, J2 Conn_01x02_Socket, J3 Conn_01x02_Socket, J4 Conn_01x02_Socket, J5 Conn_01x02_Socket, SW2 SW_Push, SW3 SW_Push, SW4 SW_Push, SW5 SW_Push

Commit message: update
Parts:
- removed the A1 at (93.0, 55.9)
- removed the C3 at (110.7, 61.0)
- removed the SW2 at (85.9, 55.9)
- removed SW3: SW_Push, TerminalBlock:TerminalBlock_Xinya_XY308-2.54-2P_1x02_P2.54mm_Horizontal
- added A3: Pololu_Breakout_DRV8825, RoboKlask:TMC2209, F.Cu at (116.8, 53.8)
- added C1: 0.1u, Capacitor_THT:C_Axial_L3.8mm_D2.6mm_P7.50mm_Horizontal, F.Cu at (92.5, 56.9)
- added C2: 0.1u, Capacitor_THT:C_Axial_L3.8mm_D2.6mm_P7.50mm_Horizontal, F.Cu at (116.8, 57.1)
- added R1: 1k, Resistor_THT:R_Box_L8.4mm_W2.5mm_P5.08mm, F.Cu at (127.0, 38.1)
- A2: value Pololu_Breakout_DRV8825 -> Breakout_TMC2209; footprint Module:Pololu_Breakout-16_15.2x20.3mm -> RoboKlask:TMC2209
- moved D1 64.4 mm to (141.0, 45.0), turned to 180 degrees
- moved J3 60.8 mm to (85.1, 74.7), turned to -90 degrees
- moved J4 60.4 mm to (85.1, 81.3), turned to -90 degrees
- moved C3 58.8 mm to (144.8, 49.3), turned to -90 degrees
- moved R3 56.6 mm to (141.5, 49.3), turned to -90 degrees
- moved R2 50.8 mm to (138.4, 54.4), turned to 90 degrees
- moved C4 48.4 mm to (85.1, 49.5)
- moved J5 25.6 mm to (85.1, 54.4), turned to -90 degrees
- moved J1 19.8 mm to (85.1, 61.2), turned to -90 degrees
- moved A2 18.7 mm to (95.8, 53.8)
- moved J2 18.4 mm to (85.1, 68.1), turned to -90 degrees
- moved SW1 0.76 mm to (85.1, 35.6)
- moved SW2 0.76 mm to (85.1, 42.2)
- renumbered A3 to A1, C1 to C3, R1 to R2, R2 to R3, SW4 to SW1, SW5 to SW2
Connections:
- A1 pad 15: /M0 -> unconnected-(A1-D0/RX-Pad15)
- A1 pad 16: /M1 -> unconnected-(A1-D1/TX-Pad16)
- A1 pad 17: /M2 -> /A0
- A1 pad 19: /MY_STEP -> /MCU2TMC
- A1 pad 20: /MY_DIR -> /TMC2MCU
- A1 pad 21: unconnected-(A3-D6-Pad21) -> /MY_STEP
- A1 pad 22: unconnected-(A3-D7-Pad22) -> /MY_DIR
- A1 pad 23: /MX_STEP -> /DIAG_Y
- A1 pad 24: /MX_DIR -> /MX_STEP
- A1 pad 25: /A0 -> /MX_DIR
- A1 pad 26: unconnected-(A3-D11-Pad26) -> /DIAG_X
- A1 pad 27: /SW_A -> /SW_Y
- A1 pad 28: /SW_B -> /SW_X
- A1 pad 31: /SW_Y -> unconnected-(A1-SDA/D20-Pad31)
- A1 pad 32: /SW_X -> unconnected-(A1-SCL/D21-Pad32)
- A1 pad 5: unconnected-(A3-+5V-Pad5) -> /5V
- A2 pad 10: /M0 -> GND
- A2 pad 11: /M1 -> GND
- A2 pad 12: /M2 -> /TMC2MCU
- A2 pad 13: /nEN -> unconnected-(A2-USART-Pad13)
- A2 pad 14: /nEN -> unconnected-(A2-CLK-Pad14)
- A2 pad 15: /MY_STEP -> /MX_STEP
- A2 pad 16: /MY_DIR -> /MX_DIR
- A2 pad 2: unconnected-(A2-~{FLT}-Pad2) -> /5V
- A2 pad 3: /MY_A2 -> /MX_A2
- A2 pad 4: /MY_A1 -> /MX_A1
- A2 pad 5: /MY_B1 -> /MX_B1
- A2 pad 6: /MY_B2 -> /MX_B2
- A2 pad 9: unconnected-(A2-~{EN}-Pad9) -> /nEN
- J3 pad 1: /MY_A1 -> /MY_A2
- J3 pad 2: /MY_A2 -> /MY_A1
Routing:
- net /5V: track 0.00 -> 98.1 mm
- net /A0: track 60.3 -> 18.8 mm
- net /M2: track 41.5 -> 0.00 mm
- net /M1: track 41.2 -> 0.00 mm
- net /M0: track 39.8 -> 0.00 mm
- net /SW_A: track 37.6 -> 0.00 mm
- net /MY_B1: track 20.9 -> 57.7 mm
- net /MY_B2: track 18.5 -> 52.8 mm
- net /TMC2MCU: track 0.00 -> 30.9 mm
- net /DIAG_X: track 0.00 -> 29.1 mm
- net /SW_B: track 28.5 -> 0.00 mm
- net /MY_A1: track 22.3 -> 48.9 mm
- net +12V: track 94.3 -> 71.4 mm
- net /MY_A2: track 24.7 -> 45.7 mm
- net /DIAG_Y: track 0.00 -> 17.1 mm, vias 0 -> 1
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
Commit message: update
Parts:
- moved C2 2.60 mm to (114.2, 57.1)
Routing:
- net /nEN: track 31.3 -> 28.9 mm
- net /MX_B2: track 30.1 -> 32.0 mm
- net /MX_A2: track 18.8 -> 20.4 mm
- net /MY_B1: track 57.7 -> 56.4 mm
- net /MX_A1: track 22.4 -> 23.7 mm
- net /5V: track 98.1 -> 97.0 mm
- net /MX_B1: track 26.5 -> 27.1 mm
- net /DIAG_Y: track 17.1 -> 16.8 mm, vias 1 -> 0
- net GND: vias 21 -> 25
Other:
- outline, holes or cut-outs redrawn

Commit message: fix pin assign
Connections:
- A2 pad 12: /TMC2MCU -> unconnected-(A2-PDN-Pad12)
- A2 pad 13: unconnected-(A2-USART-Pad13) -> /TMC2MCU
- A3 pad 12: /TMC2MCU -> unconnected-(A3-PDN-Pad12)
- A3 pad 13: unconnected-(A3-USART-Pad13) -> /TMC2MCU
Routing:
- net /TMC2MCU: track 30.9 -> 32.0 mm
Changed lines of the file:
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@@
 			(layers "*.Cu" "*.Mask")
 			(remove_unused_layers no)
-			(net "/TMC2MCU")
+			(net "unconnected-(A3-PDN-Pad12)")
 			(pinfunction "PDN_12")
-			(pintype "bidirectional")
+			(pintype "bidirectional+no_connect")
 		)
 		(pad "13" thru_hole oval
@@
 			(layers "*.Cu" "*.Mask")
 			(remove_unused_layers no)
-			(net "unconnected-(A3-USART-Pad13)")
+			(net "/TMC2MCU")
 			(pinfunction "USART_13")
-			(pintype "bidirectional+no_connect")
+			(pintype "bidirectional")
 		)
 		(pad "14" thru_hole oval
@@
 			(layers "*.Cu" "*.Mask")
 			(remove_unused_layers no)
-			(net "/TMC2MCU")
+			(net "unconnected-(A2-PDN-Pad12)")
 			(pinfunction "PDN_12")
-			(pintype "bidirectional")
+			(pintype "bidirectional+no_connect")
 		)
 		(pad "13" thru_hole oval
@@
 			(layers "*.Cu" "*.Mask")
 			(remove_unused_layers no)
-			(net "unconnected-(A2-USART-Pad13)")
+			(net "/TMC2MCU")
 			(pinfunction "USART_13")
-			(pintype "bidirectional+no_connect")
+			(pintype "bidirectional")
 		)
 		(pad "14" thru_hole oval
@@
 	)
 	(segment
-		(start 125.476 42.672)
-		(end 115.824 42.672)
+		(start 115.062 41.91)
+		(end 115.062 40.386)
 		(width 0.2)
 		(layer "B.Cu")
@@
 	(segment
 		(start 127 38.1)
-		(end 127 41.148)
+		(end 124.46 40.64)
 		(width 0.2)
 		(layer "B.Cu")
@@
 	)
 	(segment
-		(start 115.062 41.91)
-		(end 115.062 40.386)
+		(start 115.824 42.672)
+		(end 115.062 41.91)
 		(width 0.2)
 		(layer "B.Cu")
@@
 	)
 	(segment
-		(start 127 41.148)
-		(end 125.476 42.672)
+		(start 114.554 39.878)
+		(end 104.648 39.878)
 		(width 0.2)
 		(layer "B.Cu")
@@
 	)
 	(segment
-		(start 107.188 39.878)
-		(end 105.918 41.148)
+		(start 124.46 41.148)
+		(end 122.936 42.672)
 		(width 0.2)
 		(layer "B.Cu")
@@
 	)
 	(segment
-		(start 115.824 42.672)
-		(end 115.062 41.91)
+		(start 124.46 40.64)
+		(end 124.46 41.148)
 		(width 0.2)
 		(layer "B.Cu")
@@
 	)
 	(segment
-		(start 115.062 40.386)
-		(end 114.554 39.878)
+		(start 122.936 42.672)
+		(end 115.824 42.672)
 		(width 0.2)
 		(layer "B.Cu")
@@
 	)
 	(segment
-		(start 114.554 39.878)
-		(end 107.188 39.878)
+		(start 104.648 39.878)
+		(end 103.378 41.148)
+		(width 0.2)
+		(layer "B.Cu")
+		(net "/TMC2MCU")
+	)
+	(segment
+		(start 115.062 40.386)
+		(end 114.554 39.878)
 		(width 0.2)
 		(layer "B.Cu")

Commit message: update ver
Other:
- board text added: "RoboKlask v0.2.0 by motty"
- board text removed: "CoreXY 3.3V v0.1.0 by motty"
