File: Klask_PCB.kicad_sch (KiCad schematic)
At the start: 10 parts, among them SW1 SW_Push_SPDT

Commit message: update
Parts:
- added J1, J2, J3, J4: Conn_01x02_Socket, TerminalBlock:TerminalBlock_Xinya_XY308-2.54-2P_1x02_P2.54mm_Horizontal, symbol Connector:Conn_01x02_Socket
- added R3, R4: 1k, Resistor_THT:R_Box_L8.4mm_W2.5mm_P5.08mm, symbol Device:R
- added SW2, SW3: SW_Push_SPDT, TerminalBlock:TerminalBlock_Xinya_XY308-2.54-2P_1x02_P2.54mm_Horizontal, symbol Switch:SW_Push_SPDT
Connections:
- net GND: now also SW2.3 (C), SW3.3 (C)
- net MX_A1: now also J1.1 (Pin_1)
- net MX_A2: now also J1.2 (Pin_2)
- net MX_B1: now also J2.1 (Pin_1)
- net MX_B2: now also J2.2 (Pin_2)
- net MY_A1: now also J3.1 (Pin_1)
- net MY_A2: now also J3.2 (Pin_2)
- net MY_B1: now also J4.1 (Pin_1)
- net MY_B2: now also J4.2 (Pin_2)
- net SW_X: now reaches A3.26 (D11)
- net SW_X: now also R3.1
- net SW_Y: now reaches A3.27 (D12)
- net SW_Y: now also R4.1
- net 3V3: now reaches A3.4 (3V3)
- new net: R4.2, SW3.2 (B)
- new net: R3.2, SW2.2 (B)

Commit message: update
Parts:
- removed R3, R4: 1k, Resistor_THT:R_Box_L8.4mm_W2.5mm_P5.08mm, symbol Device:R
- removed SW1, SW2, SW3: SW_Push_SPDT, TerminalBlock:TerminalBlock_Xinya_XY308-2.54-2P_1x02_P2.54mm_Horizontal, symbol Switch:SW_Push_SPDT
- added SW2, SW3, SW4, SW5, SW6: SW_Push, TerminalBlock:TerminalBlock_Xinya_XY308-2.54-2P_1x02_P2.54mm_Horizontal, symbol Switch:SW_Push
- D1: footprint LED_THT:LED_D2.0mm_W4.8mm_H2.5mm_FlatTop -> LED_THT:LED_D3.0mm
- R1: value 3.3K -> 510
- R2: value 1K -> 180
Connections:
- net +12V: now also SW6.2
- net GND: now also SW2.2, SW3.2, SW4.2, SW5.2
- net MX_A1: now also J1.2 (Pin_2); no longer J1.1 (Pin_1)
- net MX_A2: now also J1.1 (Pin_1); no longer J1.2 (Pin_2)
- net MY_B1: now also J4.2 (Pin_2); no longer J4.1 (Pin_1)
- net MY_B2: now also J4.1 (Pin_1); no longer J4.2 (Pin_2)
- net MY_DIR: now also A3.20 (D5); no longer A3.19 (D4)
- net MY_STEP: now also A3.19 (D4); no longer A3.18 (D3)
- net SW_X: now also A3.31 (SDA/A4), SW4.1; no longer A3.26 (D11)
- net SW_Y: now also A3.32 (SCL/A5), SW5.1; no longer A3.27 (D12)
- net nEN: now also A3.18 (D3); no longer A3.22 (D7)
- net v_motor: now also SW6.1
- net SW_B: now reaches A3.28 (D13)
- net SW_B: now also SW3.1
- new net SW_A: A3.27 (D12), SW2.1
Other:
- note added: "0.015^2*510=0.11(W)"
- note added: "LED: 2V, 15mA(0.015A) (12-2)/0.015=666(Ohm)"
- note added: "V(A0): 2.6 = (12-2) * x / (x+y) x:x+y=26:100=173:666 x: 180, y: 510"
- note removed: "12 * 1/(3.3+1) = 2.79"

Commit message: update
Parts:
- removed SW6: SW_Push, TerminalBlock:TerminalBlock_Xinya_XY308-2.54-2P_1x02_P2.54mm_Horizontal, symbol Switch:SW_Push
- added J5: Conn_01x02_Socket, TerminalBlock:TerminalBlock_Xinya_XY308-2.54-2P_1x02_P2.54mm_Horizontal, symbol Connector:Conn_01x02_Socket
Connections:
- net v_motor is gone; now on net +12V: A1.8 (VMOT), A2.8 (VMOT), C3.1, C4.1, R1.1
- net +12V: now also J5.1 (Pin_1)
- net GND: now also J5.2 (Pin_2)
- net SW_X: now also A3.32 (SCL/A5); no longer A3.31 (SDA/A4)
- net SW_Y: now also A3.31 (SDA/A4); no longer A3.32 (SCL/A5)
Changed lines of the file:
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@@
+	)
+	(junction
+		(at 233.68 54.61)
+		(diameter 0)
+		(color 0 0 0 0)
 	)
 	(junction
@@
 	(wire
 		(pts
+			(xy 236.22 54.61) (xy 236.22 52.07)
+		)
+		(stroke
+			(width 0)
+			(type default)
+		)
+	)
+	(wire
+		(pts
 			(xy 162.56 129.54) (xy 163.83 129.54)
 		)
@@
 	(wire
 		(pts
+			(xy 233.68 54.61) (xy 233.68 64.77)
+		)
+		(stroke
+			(width 0)
+			(type default)
+		)
+	)
+	(wire
+		(pts
 			(xy 58.42 177.8) (xy 60.96 177.8)
 		)
@@
 	(wire
 		(pts
-			(xy 243.84 52.07) (xy 248.92 52.07)
-		)
-		(stroke
-			(width 0)
-			(type default)
-		)
-	)
-	(wire
-		(pts
 			(xy 83.82 109.22) (xy 83.82 107.95)
 		)
@@
 	(wire
 		(pts
-			(xy 248.92 52.07) (xy 248.92 46.99)
-		)
-		(stroke
-			(width 0)
-			(type default)
-		)
-	)
-	(wire
-		(pts
 			(xy 69.85 66.04) (xy 71.12 66.04)
 		)
@@
 	(wire
 		(pts
-			(xy 233.68 52.07) (xy 233.68 64.77)
+			(xy 233.68 52.07) (xy 233.68 54.61)
 		)
 		(stroke
@@
 		)
 	)
+	(label "SW_Y"
+		(at 97.79 96.52 0)
+		(effects
+			(font
+				(size 1.27 1.27)
+			)
+			(justify left bottom)
+		)
+	)
 	(label "MX_A2"
 		(at 180.34 55.88 0)
@@
 		)
 	)
-	(label "SW_X"
-		(at 97.79 96.52 0)
-		(effects
-			(font
-				(size 1.27 1.27)
-			)
-			(justify left bottom)
-		)
-	)
 	(label "MY_B2"
 		(at 116.84 157.48 180)
@@
 		)
 	)
-	(label "SW_Y"
-		(at 97.79 99.06 0)
-		(effects
-			(font
-				(size 1.27 1.27)
-			)
-			(justify left bottom)
-		)
-	)
 	(label "M0"
 		(at 69.85 63.5 180)
@@
 		)
 	)
+	(label "SW_X"
+		(at 97.79 99.06 0)
+		(effects
+			(font
+				(size 1.27 1.27)
+			)
+			(justify left bottom)
+		)
+	)
 	(label "MY_DIR"
 		(at 69.85 76.2 180)
@@
 			)
 			(justify left bottom)
+		)
+	)
+	(symbol
+		(lib_id "power:GND")
+		(at 236.22 54.61 90)
+		(unit 1)
+		(exclude_from_sim no)
+		(in_bom yes)
+		(on_board yes)
+		(dnp no)
+		(fields_autoplaced yes)
+		(property "Reference" "#PWR012"
+			(at 242.57 54.61 0)
+			(effects
+				(font
+					(size 1.27 1.27)
+				)
+				(hide yes)
+			)
+		)
+		(property "Value" "GND"
+			(at 240.03 54.6099 90)
+			(effects
+				(font
+					(size 1.27 1.27)
+				)
+				(justify right)
+			)
+		)
+		(property "Footprint" ""
+			(at 236.22 54.61 0)
+			(effects
+				(font
+					(size 1.27 1.27)
+				)
+				(hide yes)
+			)
+		)
+		(property "Datasheet" ""
+			(at 236.22 54.61 0)
+			(effects
+				(font
+					(size 1.27 1.27)
+				)
+				(hide yes)
+			)
+		)
+		(property "Description" "Power symbol creates a global label with name \"GND\" , ground"
+			(at 236.22 54.61 0)
+			(effects
+				(font
+					(size 1.27 1.27)
+				)
+				(hide yes)
+			)
+		)
+		(pin "1"
+		)
+		(instances
+			(project "Klask_PCB"
+				(path "/3be7f516-059a-41e8-b3c3-2dfacc710f71"
+					(reference "#PWR012")
+					(unit 1)
+				)
+			)
 		)
 	)
@@
 	)
 	(symbol
-		(lib_id "Switch:SW_Push")
-		(at 238.76 52.07 0)
-		(unit 1)
-		(exclude_from_sim no)
-		(in_bom yes)
-		(on_board yes)
-		(dnp no)
-		(fields_autoplaced yes)
-		(property "Reference" "SW6"
-			(at 238.76 44.45 0)
-			(effects
-				(font
-					(size 1.27 1.27)
-				)
-			)
-		)
-		(property "Value" "SW_Push"
-			(at 238.76 46.99 0)
-			(effects
-				(font
-					(size 1.27 1.27)
-				)
-			)
-		)
-		(property "Footprint" "TerminalBlock:TerminalBlock_Xinya_XY308-2.54-2P_1x02_P2.54mm_Horizontal"
-			(at 238.76 46.99 0)
-			(effects
-				(font
-					(size 1.27 1.27)
-				)
-				(hide yes)
-			)
-		)
-		(property "Datasheet" "~"
-			(at 238.76 46.99 0)
-			(effects
-				(font
-					(size 1.27 1.27)
-				)
-				(hide yes)
-			)
-		)
-		(property "Description" "Push button switch, generic, two pins"
-			(at 238.76 52.07 0)
-			(effects
-				(font
-					(size 1.27 1.27)
-				)
-				(hide yes)
-			)
-		)
-		(pin "1"
-		)
-		(pin "2"
-		)
-		(instances
-			(project "Klask_PCB"
-				(path "/3be7f516-059a-41e8-b3c3-2dfacc710f71"
-					(reference "SW6")
-					(unit 1)
-				)
-			)
-		)
-	)
-	(symbol
 		(lib_id "Connector:Conn_01x02_Socket")
 		(at 123.19 157.48 0)
@@
 	(symbol
 		(lib_id "power:+12V")
-		(at 248.92 46.99 0)
+		(at 233.68 54.61 90)
 		(unit 1)
 		(exclude_from_sim no)
@@
 		(fields_autoplaced yes)
 		(property "Reference" "#PWR01"
-			(at 248.92 50.8 0)
+			(at 237.49 54.61 0)
 			(effects
 				(font
@@
 		)
 		(property "Value" "+12V"
-			(at 248.92 41.91 0)
+			(at 232.41 52.07 90)
 			(effects
 				(font
@@
 		)
 		(property "Footprint" ""
-			(at 248.92 46.99 0)
+			(at 233.68 54.61 0)
 			(effects
 				(font
@@
 		)
 		(property "Datasheet" ""
-			(at 248.92 46.99 0)
+			(at 233.68 54.61 0)
 			(effects
 				(font
@@
 		)
 		(property "Description" "Power symbol creates a global label with name \"+12V\""
-			(at 248.92 46.99 0)
+			(at 233.68 54.61 0)
 			(effects
 				(font
@@
 					(unit 1)
 				)
+			)
+		)
+	)
+	(symbol
+		(lib_id "Connector:Conn_01x02_Socket")
+		(at 233.68 46.99 90)
+		(unit 1)
+		(exclude_from_sim no)
+		(in_bom yes)
+		(on_board yes)
+		(dnp no)
+		(fields_autoplaced yes)
+		(property "Reference" "J5"
+			(at 237.49 46.3549 90)
+			(effects
+				(font
+					(size 1.27 1.27)
+				)
+				(justify right)
+			)
+		)
+		(property "Value" "Conn_01x02_Socket"
+			(at 237.49 48.8949 90)
+			(effects
+				(font
+					(size 1.27 1.27)
+				)
+				(justify right)
+			)
+		)
+		(property "Footprint" "TerminalBlock:TerminalBlock_Xinya_XY308-2.54-2P_1x02_P2.54mm_Horizontal"
+			(at 233.68 46.99 0)
+			(effects
+				(font
+					(size 1.27 1.27)
+				)
+				(hide yes)
+			)
+		)
+		(property "Datasheet" "~"
+			(at 233.68 46.99 0)
+			(effects
+				(font
+					(size 1.27 1.27)
+				)
+				(hide yes)
+			)
+		)
+		(property "Description" "Generic connector, single row, 01x02, script generated"
+			(at 233.68 46.99 0)
+			(effects
+				(font
+					(size 1.27 1.27)
+				)
+				(hide yes)
+			)
+		)
+		(pin "1"
+		)
+		(pin "2"
+		)
+		(instances
+			(project "Klask_PCB"
+				(path "/3be7f516-059a-41e8-b3c3-2dfacc710f71"
+					(reference "J5")
+					(unit 1)
+				)
