File: Klask_PCB.kicad_sch (KiCad schematic)
At the start: 18 parts, among them J1 Conn_01x02_Socket, J2 Conn_01x02_Socket, J3 Conn_01x02_Socket, J4 Conn_01x02_Socket, J5 Conn_01x02_Socket, SW2 SW_Push, SW3 SW_Push, SW4 SW_Push, SW5 SW_Push

Commit message: update
Parts:
- removed A1, A2: Pololu_Breakout_DRV8825, Module:Pololu_Breakout-16_15.2x20.3mm, symbol Driver_Motor:Pololu_Breakout_DRV8825
- removed C3: 100u, Capacitor_THT:CP_Radial_D5.0mm_P2.50mm, symbol Device:C_Polarized
- removed SW2, SW3: SW_Push, TerminalBlock:TerminalBlock_Xinya_XY308-2.54-2P_1x02_P2.54mm_Horizontal, symbol Switch:SW_Push
- added A2: Breakout_TMC2209, RoboKlask:TMC2209, symbol roboklask:TMC2209
- added A3: Pololu_Breakout_DRV8825, RoboKlask:TMC2209, symbol roboklask:TMC2209
- added C1, C2: 0.1u, Capacitor_THT:C_Axial_L3.8mm_D2.6mm_P7.50mm_Horizontal, symbol Device:C
- added R1: 1k, Resistor_THT:R_Box_L8.4mm_W2.5mm_P5.08mm, symbol Device:R
- A1: renamed from A3; footprint Module:Arduino_UNO_R3 -> RoboKlask:Arduino_UNO_Q
- renumbered C1 to C3, R1 to R2, R2 to R3, SW4 to SW1, SW5 to SW2
Connections:
- net M2 is gone; now on net A0: A1.17 (D2)
- net SW_A is gone; now on net SW_Y: A1.27 (D12)
- net SW_B is gone; now on net SW_X: A1.28 (D13)
- net +12V: now also A2.8 (VMOT), A3.8 (VMOT)
- net A0: no longer A1.25 (D10)
- net GND: now also A2.1 (GND), A2.10 (MS1), A2.11 (MS2), A2.7 (GND), A3.1 (GND), A3.11 (MS2), A3.7 (GND), C1.2, C2.2
- net MX_A1: now also A2.4 (A1)
- net MX_A2: now also A2.3 (A2)
- net MX_B1: now also A2.5 (B1)
- net MX_B2: now also A2.6 (B2)
- net MX_DIR: now also A1.25 (D10), A2.16 (DIR); no longer A1.24 (D9)
- net MX_STEP: now also A1.24 (D9), A2.15 (STEP); no longer A1.23 (D8)
- net MY_A1: now also J3.2 (Pin_2), A3.4 (A1); no longer J3.1 (Pin_1)
- net MY_A2: now also J3.1 (Pin_1), A3.3 (A2); no longer J3.2 (Pin_2)
- net MY_B1: now also A3.6 (B2)
- net MY_B2: now also A3.5 (B1)
- net MY_DIR: now also A1.22 (D7), A3.16 (DIR); no longer A1.20 (D5)
- net MY_STEP: now also A1.21 (D6), A3.15 (STEP); no longer A1.19 (D4)
- net SW_X: no longer A1.32 (SCL/A5)
- net SW_Y: no longer A1.31 (SDA/A4)
- net nEN: now also A2.9 (~{EN}), A3.9 (~{EN})
- net DIAG_X: now reaches A1.26 (D11)
- net DIAG_X: now also A2.18 (DIAG)
- net 5V: now reaches A1.5 (+5V)
- net 5V: now also A2.2 (5V), A3.10 (MS1), A3.2 (5V), C1.1, C2.1
- net M0: no longer names the net of A1.15 (D0/RX)
- net M1: no longer names the net of A1.16 (D1/TX)
- new net DIAG_Y: A1.23 (D8), A3.18 (DIAG)
- new net MCU2TMC: A1.19 (D4), R1.2
- new net TMC2MCU: A1.20 (D5), A2.12 (PDN), A3.12 (PDN), R1.1
- no-connect marks 0 -> 6

Commit message: fix pin assign
Connections:
- net TMC2MCU: now also A2.13 (USART), A3.13 (USART); no longer A2.12 (PDN), A3.12 (PDN)
Changed lines of the file:
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@@
-	)
-	(no_connect
-		(at 157.48 58.42)
 	)
 	(no_connect
@@
 	)
 	(no_connect
+		(at 157.48 55.88)
+	)
+	(no_connect
 		(at 71.12 66.04)
 	)
 	(no_connect
-		(at 157.48 105.41)
+		(at 157.48 102.87)
 	)
 	(wire
@@
 	(wire
 		(pts
+			(xy 157.48 55.88) (xy 158.75 55.88)
+		)
+		(stroke
+			(width 0)
+			(type default)
+		)
+	)
+	(wire
+		(pts
 			(xy 156.21 66.04) (xy 158.75 66.04)
 		)
@@
 	(wire
 		(pts
-			(xy 149.86 102.87) (xy 158.75 102.87)
-		)
-		(stroke
-			(width 0)
-			(type default)
-		)
-	)
-	(wire
-		(pts
 			(xy 88.9 107.95) (xy 86.36 107.95)
 		)
@@
 	(wire
 		(pts
+			(xy 147.32 58.42) (xy 158.75 58.42)
+		)
+		(stroke
+			(width 0)
+			(type default)
+		)
+	)
+	(wire
+		(pts
 			(xy 236.22 54.61) (xy 236.22 52.07)
 		)
@@
 	(wire
 		(pts
-			(xy 157.48 58.42) (xy 158.75 58.42)
-		)
-		(stroke
-			(width 0)
-			(type default)
-		)
-	)
-	(wire
-		(pts
 			(xy 223.52 91.44) (xy 223.52 95.25)
 		)
@@
 	(wire
 		(pts
-			(xy 147.32 55.88) (xy 158.75 55.88)
-		)
-		(stroke
-			(width 0)
-			(type default)
-		)
-	)
-	(wire
-		(pts
 			(xy 180.34 68.58) (xy 179.07 68.58)
 		)
@@
 	(wire
 		(pts
+			(xy 157.48 102.87) (xy 158.75 102.87)
+		)
+		(stroke
+			(width 0)
+			(type default)
+		)
+	)
+	(wire
+		(pts
 			(xy 180.34 63.5) (xy 179.07 63.5)
 		)
@@
 	(wire
 		(pts
-			(xy 157.48 105.41) (xy 158.75 105.41)
-		)
-		(stroke
-			(width 0)
-			(type default)
-		)
-	)
-	(wire
-		(pts
 			(xy 227.33 58.42) (xy 233.68 58.42)
 		)
@@
 		(pts
 			(xy 50.8 73.66) (xy 50.8 76.2)
+		)
+		(stroke
+			(width 0)
+			(type default)
+		)
+	)
+	(wire
+		(pts
+			(xy 149.86 105.41) (xy 158.75 105.41)
 		)
 		(stroke
@@
 		)
 	)
-	(label "TMC_PDN"
-		(at 149.86 102.87 180)
-		(effects
-			(font
-				(size 1.27 1.27)
-			)
-			(justify right bottom)
-		)
-	)
 	(label "MY_A1"
 		(at 116.84 154.94 180)
@@
 		)
 	)
-	(label "TMC_PDN"
-		(at 147.32 55.88 180)
-		(effects
-			(font
-				(size 1.27 1.27)
-			)
-			(justify right bottom)
-		)
-	)
 	(label "MY_STEP"
 		(at 69.85 78.74 180)
@@
 		)
 	)
+	(label "TMC_PDN"
+		(at 147.32 58.42 180)
+		(effects
+			(font
+				(size 1.27 1.27)
+			)
+			(justify right bottom)
+		)
+	)
 	(label "MX_DIR"
 		(at 69.85 88.9 180)
@@
 		)
 	)
+	(label "TMC_PDN"
+		(at 149.86 105.41 180)
+		(effects
+			(font
+				(size 1.27 1.27)
+			)
+			(justify right bottom)
+		)
+	)
